File: bak.kicad_pcb (KiCad board)
At the start: 2 copper layers, 50 x 52 mm, 69 parts, among them CON1 IR_RECIEVER, CON2 HALL_SENSOR1, CON3 HALL_SENSOR2, CON4 SWD, IC1 A3G4250DTR, IC2 MCP112T-195I_TT, IC3 RN4871-V_RM140, IC4 Akcelerometr MC3479, J1 USB_B_Micro, J2 Conn_01x02_MountingPin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

Commit message: FINAL VER2
Routing:
- net GND: track 368.3 -> 373.9 mm
- net +3.3VA: track 306.6 -> 307.6 mm
Changed lines of the file:
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@@
     (thickness 1.6)
     (drawings 16)
-    (tracks 1066)
+    (tracks 1076)
     (zones 0)
     (modules 69)
@@
   )
   (setup
-    (last_trace_width 0.2)
+    (last_trace_width 0.25)
     (user_trace_width 0.2)
     (user_trace_width 0.3)
@@
       (effects (font (size 1 1) (thickness 0.15)))
     )
-    (fp_text user %R (at 0 0 90) (layer F.Fab)
-      (effects (font (size 0.4 0.4) (thickness 0.06)))
-    )
     (fp_line (start -0.8 0.4125) (end -0.8 -0.4125) (layer F.Fab) (width 0.1))
     (fp_line (start -0.8 -0.4125) (end 0.8 -0.4125) (layer F.Fab) (width 0.1))
@@
     (fp_line (start 1.65 -0.73) (end 1.65 0.73) (layer F.CrtYd) (width 0.05))
     (fp_line (start 1.65 0.73) (end -1.65 0.73) (layer F.CrtYd) (width 0.05))
+    (fp_text user %R (at 0 0 90) (layer F.Fab)
+      (effects (font (size 0.4 0.4) (thickness 0.06)))
+    )
     (pad 2 smd roundrect (at 0.9125 0 270) (size 0.975 0.95) (layers F.Cu F.Paste F.Mask) (roundrect_rratio 0.25)
       (net 53 /USB+))
@@
       (effects (font (size 1 1) (thickness 0.15)) (justify mirror))
     )
-    (fp_text user %R (at 0 0 270) (layer B.Fab)
-      (effects (font (size 0.4 0.4) (thickness 0.06)) (justify mirror))
-    )
     (fp_line (start -0.8 -0.4125) (end -0.8 0.4125) (layer B.Fab) (width 0.1))
     (fp_line (start -0.8 0.4125) (end 0.8 0.4125) (layer B.Fab) (width 0.1))
@@
     (fp_line (start 1.65 0.73) (end 1.65 -0.73) (layer B.CrtYd) (width 0.05))
     (fp_line (start 1.65 -0.73) (end -1.65 -0.73) (layer B.CrtYd) (width 0.05))
+    (fp_text user %R (at 0 0 270) (layer B.Fab)
+      (effects (font (size 0.4 0.4) (thickness 0.06)) (justify mirror))
+    )
     (pad 2 smd roundrect (at 0.9125 0 90) (size 0.975 0.95) (layers B.Cu B.Paste B.Mask) (roundrect_rratio 0.25)
       (net 76 "Net-(R18-Pad2)"))
@@
       (effects (font (size 1.27 1.27) (thickness 0.254)))
     )
-    (fp_arc (start -0.95 -3.9) (end -0.9 -3.9) (angle 180) (layer F.SilkS) (width 0.1))
-    (fp_arc (start -0.95 -3.9) (end -1 -3.9) (angle 180) (layer F.SilkS) (width 0.1))
-    (fp_text user %R (at 0 -0.48) (layer F.Fab)
-      (effects (font (size 1.27 1.27) (thickness 0.254)))
-    )
     (fp_line (start -3.7 -2.99) (end 3.7 -2.99) (layer F.Fab) (width 0.2))
     (fp_line (start 3.7 -2.99) (end 3.7 2.99) (layer F.Fab) (width 0.2))
@@
     (fp_line (start -1 -3.9) (end -1 -3.9) (layer F.SilkS) (width 0.1))
     (fp_line (start -0.9 -3.9) (end -0.9 -3.9) (layer F.SilkS) (width 0.1))
+    (fp_arc (start -0.95 -3.9) (end -0.9 -3.9) (angle 180) (layer F.SilkS) (width 0.1))
+    (fp_arc (start -0.95 -3.9) (end -1 -3.9) (angle 180) (layer F.SilkS) (width 0.1))
+    (fp_text user %R (at 0 -0.48) (layer F.Fab)
+      (effects (font (size 1.27 1.27) (thickness 0.254)))
+    )
     (pad 5 smd rect (at 1.325 -2.865 180) (size 0.4 1.4) (layers F.Cu F.Paste F.Mask)
       (net 2 GND))
@@
     (model D:\SamacSys_PCB_Library\KiCad\SamacSys_Parts.3dshapes\PTS815_SJM_250_SMTR_LFS.stp
       (at (xyz 0 0 0))
-      (scale (xyz 1 1 1))
-      (rotate (xyz 0 0 0))
+      (scale (xyz 1.1 1 1))
+      (rotate (xyz -90 0 0))
     )
   )
@@
     (model D:\SamacSys_PCB_Library\KiCad\SamacSys_Parts.3dshapes\PTS815_SJM_250_SMTR_LFS.stp
       (at (xyz 0 0 0))
-      (scale (xyz 1 1 1))
-      (rotate (xyz 0 0 0))
+      (scale (xyz 1.1 1 1))
+      (rotate (xyz -90 0 0))
     )
   )
@@
   (segment (start 86.19499 69.085) (end 88.25 71.14001) (width 0.3) (layer F.Cu) (net 2))
   (segment (start 85.54 69.085) (end 86.19499 69.085) (width 0.3) (layer F.Cu) (net 2))
-  (segment (start 59.71 73.63) (end 58.63 74.71) (width 0.3) (layer F.Cu) (net 2))
-  (via (at 58.82 73.94) (size 0.8) (drill 0.4) (layers F.Cu B.Cu) (net 2))
-  (via (at 58.63 76.225) (size 0.8) (drill 0.4) (layers F.Cu B.Cu) (net 2))
-  (segment (start 58.63 74.71) (end 58.63 76.225) (width 0.3) (layer B.Cu) (net 2))
   (segment (start 58.63 77.48) (end 58.71 77.56) (width 0.3) (layer F.Cu) (net 2))
-  (segment (start 58.63 76.225) (end 58.63 77.48) (width 0.3) (layer F.Cu) (net 2))
   (segment (start 55.59001 38.30001) (end 55.59001 40.95999) (width 0.3) (layer B.Cu) (net 2))
   (segment (start 54.09 36.8) (end 55.59001 38.30001) (width 0.3) (layer B.Cu) (net 2))
@@
   (segment (start 54.03 80.085002) (end 54.03 80.22) (width 0.3) (layer B.Cu) (net 2))
   (segment (start 57.890002 76.225) (end 54.03 80.085002) (width 0.3) (layer B.Cu) (net 2))
-  (segment (start 58.63 76.225) (end 57.890002 76.225) (width 0.3) (layer B.Cu) (net 2))
   (segment (start 56.6 62.964242) (end 55.259999 64.304243) (width 0.3) (layer B.Cu) (net 2))
   (segment (start 52.575 68.76) (end 52.4 68.935) (width 0.3) (layer F.Cu) (net 2))
@@
   (segment (start 55.299999 66.75) (end 55.299999 67.839999) (width 0.3) (layer B.Cu) (net 2))
   (segment (start 55.299999 67.839999) (end 55.56 68.1) (width 0.3) (layer B.Cu) (net 2))
+  (segment (start 57.935002 76.18) (end 57.890002 76.225) (width 0.3) (layer B.Cu) (net 2))
+  (via (at 59.52 73.65) (size 0.8) (drill 0.4) (layers F.Cu B.Cu) (net 2))
+  (segment (start 59.2 73.97) (end 59.52 73.65) (width 0.3) (layer B.Cu) (net 2))
+  (segment (start 59.2 73.97) (end 59.2 74.915002) (width 0.3) (layer B.Cu) (net 2))
+  (segment (start 58.56 75.86) (end 58.407501 75.707501) (width 0.3) (layer F.Cu) (net 2))
+  (segment (start 58.56 77.41) (end 58.56 75.86) (width 0.3) (layer F.Cu) (net 2))
+  (segment (start 58.71 77.56) (end 58.56 77.41) (width 0.3) (layer F.Cu) (net 2))
+  (via (at 58.407501 75.707501) (size 0.8) (drill 0.4) (layers F.Cu B.Cu) (net 2))
+  (segment (start 58.407501 75.707501) (end 57.890002 76.225) (width 0.3) (layer B.Cu) (net 2))
+  (segment (start 59.2 74.915002) (end 58.407501 75.707501) (width 0.3) (layer B.Cu) (net 2))
+  (segment (start 52.48 63.93) (end 52.48 62.58) (width 0.3) (layer F.Cu) (net 2))
+  (segment (start 55.299999 66.75) (end 52.48 63.93) (width 0.3) (layer F.Cu) (net 2))
   (segment (start 73.34 44.27) (end 73.34 44.73) (width 0.3) (layer B.Cu) (net 3))
   (segment (start 74.94 64.8625) (end 74.94 65.058) (width 0.25) (layer F.Cu) (net 3))
@@
   (segment (start 84.23 81.11) (end 84.23 80.505) (width 0.3) (layer F.Cu) (net 3))
   (segment (start 55.21 73.26) (end 55.21 74.47) (width 0.3) (layer F.Cu) (net 3))
-  (segment (start 56.215 75.475) (end 61.24 75.475) (width 0.3) (layer F.Cu) (net 3))
   (segment (start 55.21 74.47) (end 56.215 75.475) (width 0.3) (layer F.Cu) (net 3))
   (segment (start 56.215 76.79) (end 58.71 79.285) (width 0.3) (layer F.Cu) (net 3))
@@
   (segment (start 56.06 75.32) (end 56.215 75.475) (width 0.3) (layer F.Cu) (net 3))
   (segment (start 54.96 75.32) (end 56.06 75.32) (width 0.3) (layer F.Cu) (net 3))
+  (segment (start 61.24 75.475) (end 61.085 75.32) (width 0.3) (layer F.Cu) (net 3))
+  (segment (start 56.06 75.32) (end 56.22 75.32) (width 0.3) (layer F.Cu) (net 3))
+  (segment (start 56.22 75.32) (end 56.79 74.75) (width 0.3) (layer F.Cu) (net 3))
+  (segment (start 60.515 74.75) (end 61.24 75.475) (width 0.3) (layer F.Cu) (net 3))
+  (segment (start 56.79 74.75) (end 60.515 74.75) (width 0.3) (layer F.Cu) (net 3))
   (segment (start 62.7475 80.0475) (end 62.58 79.88) (width 0.3) (layer B.Cu) (net 4))
   (segment (start 67.43 74.568) (end 67.43 75.5) (width 0.2) (layer F.Cu) (net 4))
@@
   (segment (start 62.11 48.203237) (end 62.11 51.8) (width 0.2) (layer B.Cu) (net 53))
   (segment (start 61.630001 47.723238) (end 62.11 48.203237) (width 0.2) (layer B.Cu) (net 53))
-  (segment (start 60.58 43.73) (end 60.67 43.64) (width 0.2) (layer F.Cu) (net 77))
-  (segment (start 60.58 45.27) (end 60.58 43.73) (width 0.2) (layer F.Cu) (net 77))
   (via (at 65.45 56.44) (size 0.8) (drill 0.4) (layers F.Cu B.Cu) (net 54))
   (segment (start 67.43 61.58) (end 67.43 66.092) (width 0.2) (layer F.Cu) (net 54))
@@
   (segment (start 65.420001 56.410001) (end 65.45 56.44) (width 0.2) (layer B.Cu) (net 54))
   (segment (start 66.58 45.635) (end 65.420001 46.794999) (width 0.2) (layer B.Cu) (net 54))
-  (segment (start 62.57 43.64) (end 64.13 43.64) (width 0.2) (layer F.Cu) (net 76))
-  (via (at 64.13 43.64) (size 0.8) (drill 0.4) (layers F.Cu B.Cu) (net 76))
   (segment (start 72.467999 73.030001) (end 72.418 73.08) (width 0.2) (layer F.Cu) (net 55))
   (segment (start 72.418 73.08) (end 72.418 73.128) (width 0.2) (layer F.Cu) (net 55))
@@
   (segment (start 77.47 71.97) (end 77.19 71.69) (width 0.2) (layer B.Cu) (net 74))
   (segment (start 79.14 71.97) (end 77.47 71.97) (width 0.2) (layer B.Cu) (net 74))
+  (segment (start 62.57 43.64) (end 64.13 43.64) (width 0.2) (layer F.Cu) (net 76))
+  (via (at 64.13 43.64) (size 0.8) (drill 0.4) (layers F.Cu B.Cu) (net 76))
   (segment (start 66.3975 43.64) (end 66.42 43.6625) (width 0.2) (layer B.Cu) (net 76))
   (segment (start 64.13 43.64) (end 66.3975 43.64) (width 0.2) (layer B.Cu) (net 76))
+  (segment (start 60.58 43.73) (end 60.67 43.64) (width 0.2) (layer F.Cu) (net 77))
+  (segment (start 60.58 45.27) (end 60.58 43.73) (width 0.2) (layer F.Cu) (net 77))
   (zone (net 0) (net_name "") (layers F&B.Cu) (hatch edge 0.508)
     (connect_pads (clearance 0.508))
@@
     )
   )
-  (zone (net 2) (net_name GND) (layer F.Cu) (hatch edge 0.508)
+  (zone (net 2) (net_name GND) (layer B.Cu) (hatch edge 0.508)
     (connect_pads (clearance 0.508))
     (min_thickness 0.254)
@@
     (polygon
       (pts
-        (xy 114.58 25.92) (xy 107.08 93.52) (xy 33.11 90.65) (xy 48.53 23.46)
+        (xy 104.13 91.08) (xy 44.17 91.17) (xy 44.08 30.04) (xy 44.14 27) (xy 103.87 26.74)
       )
     )
   )
-  (zone (net 2) (net_name GND) (layer B.Cu) (hatch edge 0.508)
+  (zone (net 2) (net_name GND) (layer F.Cu) (hatch edge 0.508)
     (connect_pads (clearance 0.508))
     (min_thickness 0.254)
@@
     (polygon
       (pts
-        (xy 119.38 26.23) (xy 119.77 93.45) (xy 35.65 89.96) (xy 46.53 21.57)
+        (xy 106.04 24.96) (xy 105.99 92.99) (xy 42.02 92.99) (xy 41.99 25.99) (xy 42 24.95)
       )
     )
