File: bak.sch (KiCad schematic (older format))
At the start: 67 parts, among them CON1 IR_RECIEVER, CON2 HALL_SENSOR1, CON3 HALL_SENSOR2, CON4 Conn_01x03, CON5 Conn_01x03, IC1 A3G4250DTR, IC2 MCP112T-195I_TT, IC3 RN4871-V_RM140, IC4 Akcelerometr MC3479, J1 USB_B_Micro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

Commit message: update predelane piny a spi
Parts:
- removed CON5: Conn_01x03, Connector_Wire:SolderWire-0.1sqmm_1x03_P3.6mm_D0.4mm_OD1mm, symbol Connector_Generic:Conn_01x03
- CON1, CON2, CON3: footprint Connector_Wire:SolderWire-0.1sqmm_1x03_P3.6mm_D0.4mm_OD1mm -> KICAD_bak:MyConnector3
- CON4: value Conn_01x03 -> SWD; footprint Connector_Wire:SolderWire-0.1sqmm_1x03_P3.6mm_D0.4mm_OD1mm -> KICAD_bak:MyConnector3
- J2, J3: footprint Connector_Wire:SolderWire-0.1sqmm_1x02_P3.6mm_D0.4mm_OD1mm -> KICAD_bak:MyConnector2
Connections:
- net +3.3VA: no longer CON4.3 (Pin_3)
- net GND: now also CON2.2 (Pin_2), CON3.2 (Pin_2), CON4.2 (Pin_2); no longer CON2.1 (Pin_1), CON3.1 (Pin_1), CON4.1 (Pin_1)
- net GYRO_DRDY: no longer MCU1.42 (PB6)
- net GYRO_INT: no longer MCU1.34 (PA13)
- net HALL1: now also CON2.1 (Pin_1), MCU1.14 (PA4); no longer CON2.2 (Pin_2), MCU1.45 (PB8)
- net HALL2: now also CON3.1 (Pin_1), MCU1.15 (PA5); no longer CON3.2 (Pin_2), MCU1.43 (PB7)
- net IR_OUT: now also MCU1.16 (PA6); no longer MCU1.37 (PA14)
- net SPI2_CS: now also J4.2 (CD/DAT3); no longer IC4.2 (CSN)
- net SPI2_MISO: now also J4.7 (DAT0), R4.1; no longer IC4.3 (DOUT_A6)
- net SPI2_MOSI: now also J4.3 (CMD), R3.1; no longer IC4.4 (DIN_SDA)
- net SPI2_SCK: now also J4.5 (CLK); no longer IC4.1 (SCK_SCL)
- net SPI3_MISO: now also IC4.3 (DOUT_A6)
- net SPI3_MOSI: now also IC4.4 (DIN_SDA)
- net SPI3_SCK: now also IC4.1 (SCK_SCL)
- net CON1 renamed SPI3_CS2
- net SPI3_CS2: now also IC4.2 (CSN); no longer CON4.2 (Pin_2)
- net CON2 renamed I2C_SDA
- removed net SPI1_CS: J4.2 (CD/DAT3), MCU1.14 (PA4)
- removed net SPI1_MISO: J4.7 (DAT0), MCU1.16 (PA6), R4.1
- removed net SPI1_MOSI: J4.3 (CMD), MCU1.17 (PA7), R3.1
- removed net SPI1_SCK: J4.5 (CLK), MCU1.15 (PA5)
- net SPI3_CS renamed SPI3_CS1
- new net I2C_SCL: MCU1.42 (PB6)
- new net SWCLK: CON4.1 (Pin_1), MCU1.37 (PA14)
- new net SWDIO: CON4.3 (Pin_3), MCU1.34 (PA13)
Other:
- note removed: "SPI GYRO\n"
- note removed: "SPI SD\n"
- moved on the sheet: CON4
Changed lines of the file:
@@
 	3500 5900 3500 5800
 Text Label 10850 7500 1    50   ~ 0
-SPI3_CS
+SPI3_CS1
 $Comp
 L Device:D_Bridge_+A-A D2
@@
 Wire Wire Line
 	15650 2450 15650 2950
-Wire Wire Line
-	6100 2300 6650 2300
-Wire Wire Line
-	6100 2400 6150 2400
-Wire Wire Line
-	6100 3100 6700 3100
-Wire Wire Line
-	6100 3200 6150 3200
-Wire Wire Line
-	6150 2400 6150 2450
-Wire Wire Line
-	6150 3200 6150 3250
 Wire Notes Line
 	4950 1450 6600 1450
@@
 Text Notes 5050 1400 0    50   ~ 0
 Konektory pro další využití\n
-Text Label 6650 2300 2    50   ~ 0
-CON1
-Text Label 6700 3100 2    50   ~ 0
-CON2
-$Comp
-L power:+3.3V #PWR021
-U 1 1 6246BB04
-P 6550 2200
-F 0 "#PWR021" H 6550 2050 50  0001 C CNN
-F 1 "+3.3V" V 6565 2328 50  0000 L CNN
-F 2 "" H 6550 2200 50  0001 C CNN
-F 3 "" H 6550 2200 50  0001 C CNN
-	1    6550 2200
-	1    0    0    -1
-$EndComp
-$Comp
-L power:+3.3V #PWR022
-U 1 1 6246CD4D
-P 6550 3000
-F 0 "#PWR022" H 6550 2850 50  0001 C CNN
-F 1 "+3.3V" V 6565 3128 50  0000 L CNN
-F 2 "" H 6550 3000 50  0001 C CNN
-F 3 "" H 6550 3000 50  0001 C CNN
-	1    6550 3000
-	1    0    0    -1
-$EndComp
-$Comp
-L power:GND #PWR018
-U 1 1 6246F0F6
-P 6150 2450
-F 0 "#PWR018" H 6150 2200 50  0001 C CNN
-F 1 "GND" H 6155 2277 50  0001 C CNN
-F 2 "" H 6150 2450 50  0001 C CNN
-F 3 "" H 6150 2450 50  0001 C CNN
-	1    6150 2450
-	1    0    0    -1
-$EndComp
-$Comp
-L power:GND #PWR019
-U 1 1 6246E920
-P 6150 3250
-F 0 "#PWR019" H 6150 3000 50  0001 C CNN
-F 1 "GND" H 6155 3077 50  0001 C CNN
-F 2 "" H 6150 3250 50  0001 C CNN
-F 3 "" H 6150 3250 50  0001 C CNN
-	1    6150 3250
-	1    0    0    -1
-$EndComp
-$Comp
-L Connector_Generic:Conn_01x03 CON4
-U 1 1 61A74DBF
-P 5900 2300
-F 0 "CON4" H 5818 1975 50  0000 C CNN
-F 1 "Conn_01x03" H 5818 2066 50  0000 C CNN
-F 2 "Connector_Wire:SolderWire-0.1sqmm_1x03_P3.6mm_D0.4mm_OD1mm" H 5900 2300 50  0001 C CNN
-F 3 "~" H 5900 2300 50  0001 C CNN
-	1    5900 2300
-	-1   0    0    1
-$EndComp
-$Comp
-L Connector_Generic:Conn_01x03 CON5
-U 1 1 62442800
-P 5900 3100
-F 0 "CON5" H 5818 2775 50  0000 C CNN
-F 1 "Conn_01x03" H 5818 2866 50  0000 C CNN
-F 2 "Connector_Wire:SolderWire-0.1sqmm_1x03_P3.6mm_D0.4mm_OD1mm" H 5900 3100 50  0001 C CNN
-F 3 "~" H 5900 3100 50  0001 C CNN
-	1    5900 3100
-	-1   0    0    1
-$EndComp
 $Comp
 L Connector_Generic:Conn_01x03 CON1
@@
 F 0 "CON1" H 2818 3775 50  0000 C CNN
 F 1 "IR_RECIEVER" H 2818 3866 50  0000 C CNN
-F 2 "Connector_Wire:SolderWire-0.1sqmm_1x03_P3.6mm_D0.4mm_OD1mm" H 2900 4100 50  0001 C CNN
+F 2 "KICAD_bak:MyConnector3" H 2900 4100 50  0001 C CNN
 F 3 "~" H 2900 4100 50  0001 C CNN
 	1    2900 4100
@@
 F 0 "CON2" H 3168 1675 50  0000 C CNN
 F 1 "HALL_SENSOR1" H 3168 1766 50  0000 C CNN
-F 2 "Connector_Wire:SolderWire-0.1sqmm_1x03_P3.6mm_D0.4mm_OD1mm" H 3250 2000 50  0001 C CNN
+F 2 "KICAD_bak:MyConnector3" H 3250 2000 50  0001 C CNN
 F 3 "~" H 3250 2000 50  0001 C CNN
 	1    3250 2000
@@
 F 0 "CON3" H 3168 2425 50  0000 C CNN
 F 1 "HALL_SENSOR2" H 3168 2516 50  0000 C CNN
-F 2 "Connector_Wire:SolderWire-0.1sqmm_1x03_P3.6mm_D0.4mm_OD1mm" H 3250 2750 50  0001 C CNN
+F 2 "KICAD_bak:MyConnector3" H 3250 2750 50  0001 C CNN
 F 3 "~" H 3250 2750 50  0001 C CNN
 	1    3250 2750
@@
 L power:GND #PWR03
 U 1 1 62198691
-P 3450 2850
-F 0 "#PWR03" H 3450 2600 50  0001 C CNN
-F 1 "GND" H 3455 2677 50  0001 C CNN
-F 2 "" H 3450 2850 50  0001 C CNN
-F 3 "" H 3450 2850 50  0001 C CNN
-	1    3450 2850
+P 4050 2800
+F 0 "#PWR03" H 4050 2550 50  0001 C CNN
+F 1 "GND" H 4055 2627 50  0001 C CNN
+F 2 "" H 4050 2800 50  0001 C CNN
+F 3 "" H 4050 2800 50  0001 C CNN
+	1    4050 2800
 	1    0    0    -1
 $EndComp
@@
 L power:GND #PWR02
 U 1 1 61ABFC33
-P 3450 2100
-F 0 "#PWR02" H 3450 1850 50  0001 C CNN
-F 1 "GND" H 3455 1927 50  0001 C CNN
-F 2 "" H 3450 2100 50  0001 C CNN
-F 3 "" H 3450 2100 50  0001 C CNN
-	1    3450 2100
+P 4050 2100
+F 0 "#PWR02" H 4050 1850 50  0001 C CNN
+F 1 "GND" H 4055 1927 50  0001 C CNN
+F 2 "" H 4050 2100 50  0001 C CNN
+F 3 "" H 4050 2100 50  0001 C CNN
+	1    4050 2100
 	1    0    0    -1
 $EndComp
@@
 	1    0    0    -1
 $EndComp
-Text Label 4150 2750 2    50   ~ 0
-HALL2
-Text Label 4200 2000 2    50   ~ 0
+Text Label 3850 2100 2    50   ~ 0
 HALL1
-Text Notes 2550 3150 0    50   ~ 0
-https://cz.mouser.com/ProductDetail/621-AH49EZ3-G1
-Wire Wire Line
-	3450 2750 4150 2750
-Wire Wire Line
-	3450 2000 4200 2000
 Wire Notes Line
 	4950 1300 4950 4550
@@
 Wire Wire Line
 	4050 3750 4050 3650
-Wire Notes Line
-	2200 3200 4950 3200
-Wire Wire Line
-	3450 2650 3950 2650
 Wire Wire Line
 	3450 1900 3950 1900
 Wire Wire Line
-	6100 3000 6550 3000
-Wire Wire Line
-	6550 2200 6100 2200
+	6550 1950 6100 1950
 Wire Wire Line
 	16850 10600 16250 10600
@@
 F 0 "J2" H 11418 2375 50  0000 C CNN
 F 1 "Conn_01x02" H 11418 2466 50  0000 C CNN
-F 2 "Connector_Wire:SolderWire-0.1sqmm_1x02_P3.6mm_D0.4mm_OD1mm" H 11500 2700 50  0001 C CNN
+F 2 "KICAD_bak:MyConnector2" H 11500 2700 50  0001 C CNN
 F 3 "~" H 11500 2700 50  0001 C CNN
 	1    11500 2700
@@
 F 0 "J3" H 6268 11175 50  0000 C CNN
 F 1 "Conn_01x02" H 6268 11266 50  0000 C CNN
-F 2 "Connector_Wire:SolderWire-0.1sqmm_1x02_P3.6mm_D0.4mm_OD1mm" H 6350 11500 50  0001 C CNN
+F 2 "KICAD_bak:MyConnector2" H 6350 11500 50  0001 C CNN
 F 3 "~" H 6350 11500 50  0001 C CNN
 	1    6350 11500
@@
 	3900 7300 3900 7400
 Text Label 2950 7950 0    50   ~ 0
-SPI1_CS
+SPI2_CS
 Text Label 2950 8050 0    50   ~ 0
-SPI1_MOSI
+SPI2_MOSI
 Text Label 2950 8250 0    50   ~ 0
-SPI1_SCK
+SPI2_SCK
 Text Label 2950 8450 0    50   ~ 0
-SPI1_MISO
+SPI2_MISO
 $Comp
 L power:+3.3V #PWR012
@@
 SPI3_SCK
 Text Label 9950 10600 0    50   ~ 0
-SPI3_CS
-Text Label 9950 10500 0    50   ~ 0
-IR_OUT
+SPI3_CS1
 Text Label 11700 9850 3    50   ~ 0
 USB-
-Text Label 9950 11100 0    50   ~ 0
-HALL2
 Text Label 11600 9850 3    50   ~ 0
 USB+
@@
 Text Label 12300 9750 3    50   ~ 0
 SPI2_SCK
-Text Notes 9950 11000 1    50   ~ 0
-SPI GYRO\n
 Text Label 11900 9750 3    50   ~ 0
 ACC_INT2
@@
 Text Label 11500 12500 1    50   ~ 0
 DIODE1
-Text Label 9950 11400 0    50   ~ 0
-CON2
 Text Label 9950 10900 0    50   ~ 0
 SPI3_MOSI
-Text Label 12000 9750 3    50   ~ 0
-CON1
-Text Label 13500 11200 2    50   ~ 0
-SPI1_MOSI
 Text Label 9950 11200 0    50   ~ 0
 BOOT
-Text Label 13500 11300 2    50   ~ 0
-SPI1_MISO
-Text Label 9950 11000 0    50   ~ 0
-GYRO_DRDY
-Text Label 13500 11400 2    50   ~ 0
-SPI1_SCK
-Text Label 11500 9850 3    50   ~ 0
-GYRO_INT
-Text Label 13500 11500 2    50   ~ 0
-SPI1_CS
 Text Label 13500 11600 2    50   ~ 0
 MOTOR_PWM
@@
 Text Notes 13550 12050 0    50   ~ 0
 Diody pro možnou signalizaci\n
-Text Notes 13600 11550 1    50   ~ 0
-SPI SD\n
 Wire Wire Line
 	13100 10700 13500 10700
@@
 	1    0    0    -1
 $EndComp
-Text Label 9950 11300 0    50   ~ 0
-HALL1
 $Comp
 L SamacSys_Parts:STM32L4P5CET6 MCU1
@@
 $EndComp
 Text Label 16250 6050 0    50   ~ 0
-SPI2_SCK
+SPI3_SCK
 Text Label 16250 6150 0    50   ~ 0
-SPI2_CS
+SPI3_CS2
 Text Label 16250 6350 0    50   ~ 0
-SPI2_MOSI
+SPI3_MOSI
 Text Label 16250 6250 0    50   ~ 0
-SPI2_MISO
+SPI3_MISO
 Wire Wire Line
 	16950 6350 16250 6350
@@
 Wire Wire Line
 	5250 5400 4750 5400
+Wire Wire Line
+	6100 2150 6550 2150
+Wire Wire Line
+	6800 2050 6800 2200
+Wire Wire Line
+	6100 2050 6800 2050
+$Comp
+L power:GND #PWR0102
+U 1 1 62873F77
+P 6800 2200
+F 0 "#PWR0102" H 6800 1950 50  0001 C CNN
+F 1 "GND" H 6805 2027 50  0001 C CNN
+F 2 "" H 6800 2200 50  0001 C CNN
+F 3 "" H 6800 2200 50  0001 C CNN
+	1    6800 2200
+	1    0    0    -1
+$EndComp
+Text Label 6550 2150 2    50   ~ 0
+SWCLK
+Text Label 6550 1950 2    50   ~ 0
+SWDIO
+Text Label 9950 10500 0    50   ~ 0
+SWCLK
+Text Label 11500 9850 3    50   ~ 0
+SWDIO
+Text Label 9950 11000 0    50   ~ 0
+I2C_SCL
+Text Label 9950 11400 0    50   ~ 0
+I2C_SDA
+Text Label 12000 9750 3    50   ~ 0
+SPI3_CS2
+$Comp
+L Connector_Generic:Conn_01x03 CON4
+U 1 1 61A74DBF
+P 5900 2050
+F 0 "CON4" H 5818 1725 50  0000 C CNN
+F 1 "SWD" H 5818 1816 50  0000 C CNN
+F 2 "KICAD_bak:MyConnector3" H 5900 2050 50  0001 C CNN
+F 3 "~" H 5900 2050 50  0001 C CNN
+	1    5900 2050
+	-1   0    0    1
+$EndComp
+Wire Notes Line
+	2200 3200 4950 3200
+Text Notes 2550 3150 0    50   ~ 0
+https://cz.mouser.com/ProductDetail/621-AH49EZ3-G1
+Text Label 13500 11500 2    50   ~ 0
+HALL1
+Text Label 13500 11400 2    50   ~ 0
+HALL2
+Text Label 13500 11300 2    50   ~ 0
+IR_OUT
+Wire Wire Line
+	4050 2750 4050 2800
+Text Label 3800 2850 2    50   ~ 0
+HALL2
+Wire Wire Line
+	3450 2100 3850 2100
+Wire Wire Line
+	3800 2850 3450 2850
+Wire Wire Line
+	3450 2000 4050 2000
+Wire Wire Line
+	4050 2000 4050 2100
+Wire Wire Line
+	3450 2650 3950 2650
+Wire Wire Line
+	3450 2750 4050 2750
 $EndSCHEMATC

Commit message: cca predelano
Parts:
- added C23: 100n, Capacitor_SMD:C_0805_2012Metric_Pad1.18x1.45mm_HandSolder, symbol Device:C
- added SW3: SW_Push_Open, SamacSys_Parts:PTS815SJM250SMTRLFS, symbol Switch:SW_Push_Open
Connections:
- net GND: now also C23.2, SW3.1 (A)
- net BTN: now reaches MCU1.17 (PA7)
- net BTN: now also C23.1, SW3.2 (B)
Other:
- moved on the sheet: C4, R5, SW1, SW2
Changed lines of the file:
@@
 Connection ~ 9200 8300
 Connection ~ 9200 8600
-Connection ~ 8700 10800
 Connection ~ 9650 8300
 Connection ~ 9650 8600
@@
 	3400 4050 3400 4100
 Wire Wire Line
-	8350 10800 8700 10800
-Wire Wire Line
-	8350 11200 8350 11300
-Wire Wire Line
-	8500 10050 8100 10050
-Wire Wire Line
 	9200 8200 9200 8300
 Wire Wire Line
 	9200 8600 9200 8700
 Wire Wire Line
-	8700 10800 9250 10800
-Wire Wire Line
-	8700 11100 8700 11300
-Wire Wire Line
-	8900 10050 8800 10050
-Wire Wire Line
 	9650 8300 9200 8300
 Wire Wire Line
 	9650 8600 9200 8600
 Wire Wire Line
-	9300 9950 9450 9950
-Wire Wire Line
 	9300 12400 9450 12400
 Wire Wire Line
@@
 Wire Wire Line
 	10850 7100 10850 7500
-Wire Wire Line
-	9450 9950 9450 9800
-Wire Wire Line
-	9450 10150 9300 10150
-Wire Wire Line
-	9450 10300 9450 10150
 Wire Wire Line
 	9450 12400 9450 12600
@@
 Text Label 3750 4200 2    50   ~ 0
 IR_OUT
-Text Label 8100 10050 0    50   ~ 0
-BOOT
-Text Label 9250 10800 2    50   ~ 0
+Text Label 9150 10750 2    50   ~ 0
 NRST
 Text Label 10950 7500 1    50   ~ 0
@@
 $EndComp
 $Comp
-L power:+3.3V #PWR030
-U 1 1 6219EFB7
-P 9450 9800
-F 0 "#PWR030" H 9450 9650 50  0001 C CNN
-F 1 "+3.3V" H 9465 9973 50  0000 C CNN
-F 2 "" H 9450 9800 50  0001 C CNN
-F 3 "" H 9450 9800 50  0001 C CNN
-	1    9450 9800
-	1    0    0    -1
-$EndComp
-$Comp
 L power:+3.3V #PWR036
 U 1 1 61CC474F
@@
 $EndComp
 $Comp
-L power:GND #PWR023
-U 1 1 6313202C
-P 8350 11300
-F 0 "#PWR023" H 8350 11050 50  0001 C CNN
-F 1 "GND" H 8355 11127 50  0001 C CNN
-F 2 "" H 8350 11300 50  0001 C CNN
-F 3 "" H 8350 11300 50  0001 C CNN
-	1    8350 11300
-	1    0    0    -1
-$EndComp
-$Comp
 L power:GND #PWR024
 U 1 1 6286A997
@@
 F 3 "" H 9200 8700 50  0001 C CNN
 	1    9200 8700
-	1    0    0    -1
-$EndComp
-$Comp
-L power:GND #PWR025
-U 1 1 6315D41E
-P 8700 11300
-F 0 "#PWR025" H 8700 11050 50  0001 C CNN
-F 1 "GND" H 8705 11127 50  0001 C CNN
-F 2 "" H 8700 11300 50  0001 C CNN
-F 3 "" H 8700 11300 50  0001 C CNN
-	1    8700 11300
-	1    0    0    -1
-$EndComp
-$Comp
-L power:GND #PWR031
-U 1 1 6219E7A2
-P 9450 10300
-F 0 "#PWR031" H 9450 10050 50  0001 C CNN
-F 1 "GND" H 9455 10127 50  0001 C CNN
-F 2 "" H 9450 10300 50  0001 C CNN
-F 3 "" H 9450 10300 50  0001 C CNN
-	1    9450 10300
 	1    0    0    -1
 $EndComp
@@
 $EndComp
 $Comp
-L Device:R R5
-U 1 1 6218A78F
-P 8650 10050
-F 0 "R5" V 8443 10050 50  0000 C CNN
-F 1 "10k" V 8534 10050 50  0000 C CNN
-F 2 "Resistor_SMD:R_0805_2012Metric_Pad1.20x1.40mm_HandSolder" V 8580 10050 50  0001 C CNN
-F 3 "~" H 8650 10050 50  0001 C CNN
-	1    8650 10050
-	0    -1   -1   0
-$EndComp
-$Comp
 L Device:R R6
 U 1 1 621D383D
@@
 	1    14350 12600
 	-1   0    0    1
-$EndComp
-$Comp
-L Switch:SW_Push_Open SW1
-U 1 1 630D63C7
-P 8350 11000
-F 0 "SW1" V 8400 11250 50  0000 R CNN
-F 1 "SW_Push_Open" V 8300 11600 50  0000 R CNN
-F 2 "SamacSys_Parts:PTS815SJM250SMTRLFS" H 8350 11200 50  0001 C CNN
-F 3 "~" H 8350 11200 50  0001 C CNN
-	1    8350 11000
-	0    -1   -1   0
 $EndComp
 $Comp
@@
 $EndComp
 $Comp
-L Device:C C4
-U 1 1 6307F914
-P 8700 10950
-F 0 "C4" H 8815 10996 50  0000 L CNN
-F 1 "100n" H 8815 10905 50  0000 L CNN
-F 2 "Capacitor_SMD:C_0805_2012Metric_Pad1.18x1.45mm_HandSolder" H 8738 10800 50  0001 C CNN
-F 3 "~" H 8700 10950 50  0001 C CNN
-	1    8700 10950
-	1    0    0    -1
-$EndComp
-$Comp
 L Device:C C6
 U 1 1 61C213EF
@@
 	1    15150 2800
 	1    0    0    1
-$EndComp
-$Comp
-L Switch:SW_SPDT SW2
-U 1 1 621891DD
-P 9100 10050
-F 0 "SW2" H 9100 10335 50  0000 C CNN
-F 1 "SW_SPDT" H 9100 10244 50  0000 C CNN
-F 2 "SamacSys_Parts:SSSS810701" H 9100 10050 50  0001 C CNN
-F 3 "~" H 9100 10050 50  0001 C CNN
-	1    9100 10050
-	1    0    0    -1
 $EndComp
 $Comp
@@
 Wire Wire Line
 	11700 8750 11700 8600
-Wire Wire Line
-	12800 8600 12250 8600
 Connection ~ 11700 8600
 Connection ~ 12250 8600
@@
 Wire Wire Line
 	3450 2750 4050 2750
+$Comp
+L Device:C C4
+U 1 1 6307F914
+P 8600 10900
+F 0 "C4" H 8715 10946 50  0000 L CNN
+F 1 "100n" H 8715 10855 50  0000 L CNN
+F 2 "Capacitor_SMD:C_0805_2012Metric_Pad1.18x1.45mm_HandSolder" H 8638 10750 50  0001 C CNN
+F 3 "~" H 8600 10900 50  0001 C CNN
+	1    8600 10900
+	1    0    0    -1
+$EndComp
+$Comp
+L Switch:SW_Push_Open SW1
+U 1 1 630D63C7
+P 8250 10950
+F 0 "SW1" V 8300 11200 50  0000 R CNN
+F 1 "SW_Push_Open" V 8200 11550 50  0000 R CNN
+F 2 "SamacSys_Parts:PTS815SJM250SMTRLFS" H 8250 11150 50  0001 C CNN
+F 3 "~" H 8250 11150 50  0001 C CNN
+	1    8250 10950
+	0    -1   -1   0
+$EndComp
+$Comp
+L power:GND #PWR025
+U 1 1 6315D41E
+P 8600 11250
+F 0 "#PWR025" H 8600 11000 50  0001 C CNN
+F 1 "GND" H 8605 11077 50  0001 C CNN
+F 2 "" H 8600 11250 50  0001 C CNN
+F 3 "" H 8600 11250 50  0001 C CNN
+	1    8600 11250
+	1    0    0    -1
+$EndComp
+$Comp
+L power:GND #PWR023
+U 1 1 6313202C
+P 8250 11250
+F 0 "#PWR023" H 8250 11000 50  0001 C CNN
+F 1 "GND" H 8255 11077 50  0001 C CNN
+F 2 "" H 8250 11250 50  0001 C CNN
+F 3 "" H 8250 11250 50  0001 C CNN
+	1    8250 11250
+	1    0    0    -1
+$EndComp
+Wire Wire Line
+	8600 11050 8600 11250
+Wire Wire Line
+	8600 10750 9150 10750
+Wire Wire Line
+	8250 11150 8250 11250
+Wire Wire Line
+	8250 10750 8600 10750
+Connection ~ 8600 10750
+Wire Wire Line
+	12800 8600 12250 8600
+$Comp
+L Device:R R5
+U 1 1 6218A78F
+P 13400 9200
+F 0 "R5" V 13193 9200 50  0000 C CNN
+F 1 "10k" V 13284 9200 50  0000 C CNN
+F 2 "Resistor_SMD:R_0805_2012Metric_Pad1.20x1.40mm_HandSolder" V 13330 9200 50  0001 C CNN
+F 3 "~" H 13400 9200 50  0001 C CNN
+	1    13400 9200
+	0    -1   -1   0
+$EndComp
+$Comp
+L power:+3.3V #PWR030
+U 1 1 6219EFB7
+P 14200 8950
+F 0 "#PWR030" H 14200 8800 50  0001 C CNN
+F 1 "+3.3V" H 14215 9123 50  0000 C CNN
+F 2 "" H 14200 8950 50  0001 C CNN
+F 3 "" H 14200 8950 50  0001 C CNN
+	1    14200 8950
+	1    0    0    -1
+$EndComp
+Text Label 12850 9200 0    50   ~ 0
+BOOT
+Wire Wire Line
+	14200 9100 14200 8950
+Wire Wire Line
+	14050 9100 14200 9100
+Wire Wire Line
+	13650 9200 13550 9200
+Wire Wire Line
+	13250 9200 12850 9200
+Wire Wire Line
+	14200 9300 14050 9300
+Wire Wire Line
+	14200 9450 14200 9300
+$Comp
+L power:GND #PWR031
+U 1 1 6219E7A2
+P 14200 9450
+F 0 "#PWR031" H 14200 9200 50  0001 C CNN
+F 1 "GND" H 14205 9277 50  0001 C CNN
+F 2 "" H 14200 9450 50  0001 C CNN
+F 3 "" H 14200 9450 50  0001 C CNN
+	1    14200 9450
+	1    0    0    -1
+$EndComp
+$Comp
+L Switch:SW_SPDT SW2
+U 1 1 621891DD
+P 13850 9200
+F 0 "SW2" H 13850 9485 50  0000 C CNN
+F 1 "SW_SPDT" H 13850 9394 50  0000 C CNN
+F 2 "SamacSys_Parts:SSSS810701" H 13850 9200 50  0001 C CNN
+F 3 "~" H 13850 9200 50  0001 C CNN
+	1    13850 9200
+	1    0    0    -1
+$EndComp
+Text Label 9150 9550 2    50   ~ 0
+BTN
+$Comp
+L Device:C C23
+U 1 1 6285D17C
+P 8600 9700
+F 0 "C23" H 8715 9746 50  0000 L CNN
+F 1 "100n" H 8715 9655 50  0000 L CNN
+F 2 "Capacitor_SMD:C_0805_2012Metric_Pad1.18x1.45mm_HandSolder" H 8638 9550 50  0001 C CNN
+F 3 "~" H 8600 9700 50  0001 C CNN
+	1    8600 9700
+	1    0    0    -1
+$EndComp
+$Comp
+L Switch:SW_Push_Open SW3
+U 1 1 6285D182
+P 8250 9750
+F 0 "SW3" V 8300 10000 50  0000 R CNN
+F 1 "SW_Push_Open" V 8200 10350 50  0000 R CNN
+F 2 "SamacSys_Parts:PTS815SJM250SMTRLFS" H 8250 9950 50  0001 C CNN
+F 3 "~" H 8250 9950 50  0001 C CNN
+	1    8250 9750
+	0    -1   -1   0
+$EndComp
+$Comp
+L power:GND #PWR0103
+U 1 1 6285D188
+P 8600 10050
+F 0 "#PWR0103" H 8600 9800 50  0001 C CNN
+F 1 "GND" H 8605 9877 50  0001 C CNN
+F 2 "" H 8600 10050 50  0001 C CNN
+F 3 "" H 8600 10050 50  0001 C CNN
+	1    8600 10050
+	1    0    0    -1
+$EndComp
+$Comp
+L power:GND #PWR0104
+U 1 1 6285D18E
+P 8250 10050
+F 0 "#PWR0104" H 8250 9800 50  0001 C CNN
+F 1 "GND" H 8255 9877 50  0001 C CNN
+F 2 "" H 8250 10050 50  0001 C CNN
+F 3 "" H 8250 10050 50  0001 C CNN
+	1    8250 10050
+	1    0    0    -1
+$EndComp
+Wire Wire Line
+	8600 9850 8600 10050
+Wire Wire Line
+	8600 9550 9150 9550
+Wire Wire Line
+	8250 9950 8250 10050
+Wire Wire Line
+	8250 9550 8600 9550
+Connection ~ 8600 9550
+Text Label 13500 11200 2    50   ~ 0
+BTN
 $EndSCHEMATC
