File: bak.sch (KiCad schematic (older format))
At the start: 68 parts, among them CON1 IR_RECIEVER, CON2 HALL_SENSOR1, CON3 HALL_SENSOR2, CON4 SWD, IC1 A3G4250DTR, IC2 MCP112T-195I_TT, IC3 RN4871-V_RM140, IC4 Akcelerometr MC3479, J1 USB_B_Micro, J2 Conn_01x02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

Commit message: hotovo_snad
Connections:
- net I2C_SCL is gone; now on net GYRO_DRDY: MCU1.42 (PB6)
- net GYRO_INT: now also MCU1.38 (PA15)
- net SPI3_CS1: now also MCU1.43 (PB7); no longer MCU1.38 (PA15)
- net I2C_SDA: no longer names the net of MCU1.46 (PB9)
- no-connect marks 19 -> 21
Other:
- note added: "SWD konektor\n\n"
- note removed: "Konektory pro další využití\n"
- moved on the sheet: CON4
Changed lines of the file:
@@
 	3450 4750 3450 4550
-Wire Notes Line
-	3000 3350 3000 3200
 Wire Notes Line
 	7400 7950 8450 7950
@@
 	15650 2450 15650 2950
 Wire Notes Line
-	4950 1450 6600 1450
-Wire Notes Line
 	6600 1450 6600 1300
-Text Notes 5050 1400 0    50   ~ 0
-Konektory pro další využití\n
 $Comp
 L Connector_Generic:Conn_01x03 CON1
@@
 	-1   0    0    1
 $EndComp
-Text Notes 2350 3300 0    50   ~ 0
-IR přijímač\n
-Wire Notes Line
-	2200 3350 3000 3350
-$Comp
-L Connector_Generic:Conn_01x03 CON2
-U 1 1 62632C99
-P 3250 2000
-F 0 "CON2" H 3168 1675 50  0000 C CNN
-F 1 "HALL_SENSOR1" H 3168 1766 50  0000 C CNN
-F 2 "KICAD_bak:MyConnector3" H 3250 2000 50  0001 C CNN
-F 3 "~" H 3250 2000 50  0001 C CNN
-	1    3250 2000
-	-1   0    0    1
-$EndComp
-$Comp
-L Connector_Generic:Conn_01x03 CON3
-U 1 1 626324A3
-P 3250 2750
-F 0 "CON3" H 3168 2425 50  0000 C CNN
-F 1 "HALL_SENSOR2" H 3168 2516 50  0000 C CNN
-F 2 "KICAD_bak:MyConnector3" H 3250 2750 50  0001 C CNN
-F 3 "~" H 3250 2750 50  0001 C CNN
-	1    3250 2750
-	-1   0    0    1
-$EndComp
 Wire Notes Line
 	3850 1450 3850 1300
-Text Notes 2700 1400 0    50   ~ 0
+Text Notes 2550 1400 0    50   ~ 0
 Připojení Hallova senzoru\n
-$Comp
-L power:GND #PWR03
-U 1 1 62198691
-P 4050 2800
-F 0 "#PWR03" H 4050 2550 50  0001 C CNN
-F 1 "GND" H 4055 2627 50  0001 C CNN
-F 2 "" H 4050 2800 50  0001 C CNN
-F 3 "" H 4050 2800 50  0001 C CNN
-	1    4050 2800
-	1    0    0    -1
-$EndComp
-$Comp
-L power:GND #PWR02
-U 1 1 61ABFC33
-P 4050 2100
-F 0 "#PWR02" H 4050 1850 50  0001 C CNN
-F 1 "GND" H 4055 1927 50  0001 C CNN
-F 2 "" H 4050 2100 50  0001 C CNN
-F 3 "" H 4050 2100 50  0001 C CNN
-	1    4050 2100
-	1    0    0    -1
-$EndComp
-$Comp
-L power:+3.3V #PWR08
-U 1 1 6219868B
-P 3950 2650
-F 0 "#PWR08" H 3950 2500 50  0001 C CNN
-F 1 "+3.3V" V 3965 2778 50  0000 L CNN
-F 2 "" H 3950 2650 50  0001 C CNN
-F 3 "" H 3950 2650 50  0001 C CNN
-	1    3950 2650
-	1    0    0    -1
-$EndComp
-$Comp
-L power:+3.3V #PWR07
-U 1 1 61AA8ACC
-P 3950 1900
-F 0 "#PWR07" H 3950 1750 50  0001 C CNN
-F 1 "+3.3V" V 3965 2028 50  0000 L CNN
-F 2 "" H 3950 1900 50  0001 C CNN
-F 3 "" H 3950 1900 50  0001 C CNN
-	1    3950 1900
-	1    0    0    -1
-$EndComp
-Text Label 3850 2100 2    50   ~ 0
-HALL1
-Wire Notes Line
-	4950 1300 4950 4550
 Wire Notes Line
 	2200 1450 3850 1450
@@
 Wire Wire Line
 	4050 3750 4050 3650
-Wire Wire Line
-	3450 1900 3950 1900
-Wire Wire Line
-	6550 1950 6100 1950
 Wire Wire Line
 	16850 10600 16250 10600
@@
 Wire Notes Line
 	2200 13550 21850 13550
-Wire Notes Line
-	2200 1300 21850 1300
 Text Notes 14850 7950 0    50   ~ 0
 BLE MODUL RN4871-V/RM140
@@
 Wire Wire Line
 	9450 12400 9800 12400
-Wire Notes Line
-	7400 1300 7400 13550
 $Comp
 L SamacSys_Parts:ECS-160-8-36B2-CKM-TR Crystal1
@@
 Text Label 9950 10700 0    50   ~ 0
 SPI3_SCK
-Text Label 9950 10600 0    50   ~ 0
+Text Label 9950 11100 0    50   ~ 0
 SPI3_CS1
 Text Label 11700 9850 3    50   ~ 0
@@
 	13500 11300 13100 11300
 Wire Wire Line
-	10400 11300 9950 11300
-Wire Wire Line
 	13100 11400 13500 11400
-Wire Wire Line
-	10400 11400 9950 11400
 Wire Wire Line
 	13100 11500 13500 11500
@@
 Wire Wire Line
 	5250 5400 4750 5400
-Wire Wire Line
-	6100 2150 6550 2150
-Wire Wire Line
-	6800 2050 6800 2200
-Wire Wire Line
-	6100 2050 6800 2050
-$Comp
-L power:GND #PWR0102
-U 1 1 62873F77
-P 6800 2200
-F 0 "#PWR0102" H 6800 1950 50  0001 C CNN
-F 1 "GND" H 6805 2027 50  0001 C CNN
-F 2 "" H 6800 2200 50  0001 C CNN
-F 3 "" H 6800 2200 50  0001 C CNN
-	1    6800 2200
-	1    0    0    -1
-$EndComp
-Text Label 6550 2150 2    50   ~ 0
-SWCLK
-Text Label 6550 1950 2    50   ~ 0
-SWDIO
 Text Label 9950 10500 0    50   ~ 0
 SWCLK
 Text Label 11500 9850 3    50   ~ 0
 SWDIO
-Text Label 9950 11000 0    50   ~ 0
-I2C_SCL
-Text Label 9950 11400 0    50   ~ 0
-I2C_SDA
 Text Label 12000 9750 3    50   ~ 0
 SPI3_CS2
-$Comp
-L Connector_Generic:Conn_01x03 CON4
-U 1 1 61A74DBF
-P 5900 2050
-F 0 "CON4" H 5818 1725 50  0000 C CNN
-F 1 "SWD" H 5818 1816 50  0000 C CNN
-F 2 "KICAD_bak:MyConnector3" H 5900 2050 50  0001 C CNN
-F 3 "~" H 5900 2050 50  0001 C CNN
-	1    5900 2050
-	-1   0    0    1
-$EndComp
-Wire Notes Line
-	2200 3200 4950 3200
-Text Notes 2550 3150 0    50   ~ 0
-https://cz.mouser.com/ProductDetail/621-AH49EZ3-G1
 Text Label 13500 11500 2    50   ~ 0
 HALL1
@@
 Text Label 13500 11300 2    50   ~ 0
 IR_OUT
-Wire Wire Line
-	4050 2750 4050 2800
-Text Label 3800 2850 2    50   ~ 0
-HALL2
-Wire Wire Line
-	3450 2100 3850 2100
-Wire Wire Line
-	3800 2850 3450 2850
-Wire Wire Line
-	3450 2000 4050 2000
-Wire Wire Line
-	4050 2000 4050 2100
-Wire Wire Line
-	3450 2650 3950 2650
-Wire Wire Line
-	3450 2750 4050 2750
 $Comp
 L Device:C C4
@@
 Text Label 13500 11200 2    50   ~ 0
 BTN
+Text Label 9950 10600 0    50   ~ 0
+GYRO_INT
+Text Label 9950 11000 0    50   ~ 0
+GYRO_DRDY
+NoConn ~ 10400 11300
+NoConn ~ 10400 11400
+Wire Wire Line
+	3450 2750 4050 2750
+Wire Wire Line
+	3450 2650 3950 2650
+Wire Wire Line
+	4050 2000 4050 2100
+Wire Wire Line
+	3450 2000 4050 2000
+Wire Wire Line
+	3800 2850 3450 2850
+Wire Wire Line
+	3450 2100 3850 2100
+Text Label 3800 2850 2    50   ~ 0
+HALL2
+Wire Wire Line
+	4050 2750 4050 2800
+Text Notes 2550 3150 0    50   ~ 0
+https://cz.mouser.com/ProductDetail/621-AH49EZ3-G1
+Wire Notes Line
+	2200 3200 4950 3200
+$Comp
+L Connector_Generic:Conn_01x03 CON4
+U 1 1 61A74DBF
+P 5750 2650
+F 0 "CON4" H 5668 2325 50  0000 C CNN
+F 1 "SWD" H 5668 2416 50  0000 C CNN
+F 2 "KICAD_bak:MyConnector3" H 5750 2650 50  0001 C CNN
+F 3 "~" H 5750 2650 50  0001 C CNN
+	1    5750 2650
+	-1   0    0    1
+$EndComp
+Text Label 6400 2550 2    50   ~ 0
+SWDIO
+Text Label 6400 2750 2    50   ~ 0
+SWCLK
+$Comp
+L power:GND #PWR0102
+U 1 1 62873F77
+P 6650 2800
+F 0 "#PWR0102" H 6650 2550 50  0001 C CNN
+F 1 "GND" H 6655 2627 50  0001 C CNN
+F 2 "" H 6650 2800 50  0001 C CNN
+F 3 "" H 6650 2800 50  0001 C CNN
+	1    6650 2800
+	1    0    0    -1
+$EndComp
+Wire Wire Line
+	5950 2650 6650 2650
+Wire Wire Line
+	6650 2650 6650 2800
+Wire Wire Line
+	5950 2750 6400 2750
+Wire Notes Line
+	7400 1300 7400 13550
+Wire Wire Line
+	6400 2550 5950 2550
+Wire Wire Line
+	3450 1900 3950 1900
+Wire Notes Line
+	4950 1300 4950 4550
+Text Label 3850 2100 2    50   ~ 0
+HALL1
+$Comp
+L power:+3.3V #PWR07
+U 1 1 61AA8ACC
+P 3950 1900
+F 0 "#PWR07" H 3950 1750 50  0001 C CNN
+F 1 "+3.3V" V 3965 2028 50  0000 L CNN
+F 2 "" H 3950 1900 50  0001 C CNN
+F 3 "" H 3950 1900 50  0001 C CNN
+	1    3950 1900
+	1    0    0    -1
+$EndComp
+$Comp
+L power:+3.3V #PWR08
+U 1 1 6219868B
+P 3950 2650
+F 0 "#PWR08" H 3950 2500 50  0001 C CNN
+F 1 "+3.3V" V 3965 2778 50  0000 L CNN
+F 2 "" H 3950 2650 50  0001 C CNN
+F 3 "" H 3950 2650 50  0001 C CNN
+	1    3950 2650
+	1    0    0    -1
+$EndComp
+$Comp
+L power:GND #PWR02
+U 1 1 61ABFC33
+P 4050 2100
+F 0 "#PWR02" H 4050 1850 50  0001 C CNN
+F 1 "GND" H 4055 1927 50  0001 C CNN
+F 2 "" H 4050 2100 50  0001 C CNN
+F 3 "" H 4050 2100 50  0001 C CNN
+	1    4050 2100
+	1    0    0    -1
+$EndComp
+$Comp
+L power:GND #PWR03
+U 1 1 62198691
+P 4050 2800
+F 0 "#PWR03" H 4050 2550 50  0001 C CNN
+F 1 "GND" H 4055 2627 50  0001 C CNN
+F 2 "" H 4050 2800 50  0001 C CNN
+F 3 "" H 4050 2800 50  0001 C CNN
+	1    4050 2800
+	1    0    0    -1
+$EndComp
+$Comp
+L Connector_Generic:Conn_01x03 CON3
+U 1 1 626324A3
+P 3250 2750
+F 0 "CON3" H 3168 2425 50  0000 C CNN
+F 1 "HALL_SENSOR2" H 3168 2516 50  0000 C CNN
+F 2 "KICAD_bak:MyConnector3" H 3250 2750 50  0001 C CNN
+F 3 "~" H 3250 2750 50  0001 C CNN
+	1    3250 2750
+	-1   0    0    1
+$EndComp
+$Comp
+L Connector_Generic:Conn_01x03 CON2
+U 1 1 62632C99
+P 3250 2000
+F 0 "CON2" H 3168 1675 50  0000 C CNN
+F 1 "HALL_SENSOR1" H 3168 1766 50  0000 C CNN
+F 2 "KICAD_bak:MyConnector3" H 3250 2000 50  0001 C CNN
+F 3 "~" H 3250 2000 50  0001 C CNN
+	1    3250 2000
+	-1   0    0    1
+$EndComp
+Wire Notes Line
+	2200 3350 3000 3350
+Text Notes 2350 3300 0    50   ~ 0
+IR přijímač\n
+Wire Notes Line
+	3000 3350 3000 3200
+Wire Notes Line
+	4950 1450 6600 1450
+Wire Notes Line
+	2200 1300 21850 1300
+Text Notes 5600 1500 0    50   ~ 0
+SWD konektor\n\n
 $EndSCHEMATC

Commit message: snad final, zony, upraveny 3D modely, upraveny tlacitko
Parts:
- removed C23: 100n, Capacitor_SMD:C_0805_2012Metric_Pad1.18x1.45mm_HandSolder, symbol Device:C
- added R17: 10k, Resistor_SMD:R_0805_2012Metric_Pad1.20x1.40mm_HandSolder, symbol Device:R
- Q1: footprint DPAK3-CASE-369AS -> SamacSys_Parts:DPAK3-CASE-369AS
Connections:
- net +3.3VA: now also R17.2
- net BTN: now also R17.1
- no-connect marks 21 -> 20
Other:
- note removed: "Bylo by vhodné připad proudovou ochranu\nsloženou z PTC pojistky a transilu"
- note removed: "Je vhodné stínění USB připojit\nferitovou perlou/korálkem na zem"
- note removed: "Je vážný důvod mít jeden senzor na SPI a druhý na I2C?\nPřípadně bych asi očekával, že data z akcelerometru budou\npotřeba s vyšší frekvencí a přesto je na pomalejší sběrnici"
- note removed: "Obecné:\n- Pokud má zapojení jen jednu zem, pak se běžně nepoužívá u značky label GND\n- Schéma by možná bylo lepší pojmout hierarchicky (oddělených částí má docela dost)\n- V případě flat schématu by bylo lepší boxy rozmítit, nějak hezčeji a ne je jen rozházet po prostoru\n- Neexistuje zde jednost v zápisu hodnot: 2k5 vs 2.7k, objevuje se jich zde několik"
- note removed: "Užitečné připomínky"
- note removed: "Účel konektoru by měl být napsán v hodnotě,\npřípadně vedle značky, není vhodné jej dávat\ndo reference, přestože v rámci generování BOMu\nto dává více smysl, pro generování výstupních\npodkladů to naopak smysl nedává"
- moved on the sheet: SW3
Changed lines of the file:
@@
 Sheet 1 1
 Title "Carrera Car"
-Date "2022-03-22"
-Rev ""
+Date "2022-05-08"
+Rev "Version 2"
 Comp ""
 Comment1 "Vojtěch Šíma, Fakulta informačních technologií  VUT v Brně"
@@
 NoConn ~ -350 1300
 NoConn ~ 3900 5600
-NoConn ~ 4800 14350
 Wire Wire Line
 	3900 5400 4300 5400
@@
 Wire Notes Line
 	15350 4050 15350 3900
-Text Notes 6300 15000 0    50   ~ 0
-Účel konektoru by měl být napsán v hodnotě,\npřípadně vedle značky, není vhodné jej dávat\ndo reference, přestože v rámci generování BOMu\nto dává více smysl, pro generování výstupních\npodkladů to naopak smysl nedává
 Text Notes 2250 6500 0    50   ~ 0
 USB https://www.mouser.co.uk/ProductDetail/GCT/USB3065-30-00-A?qs=iLbezkQI%252Bshlw4HeJLlWGw%3D%3D
@@
 Text Notes 2300 4700 0    50   ~ 0
 Micro USB a ESD protekce\n
-Text Notes 2850 15600 0    50   ~ 0
-Je vhodné stínění USB připojit\nferitovou perlou/korálkem na zem
 Text Notes 2350 4500 0    50   ~ 0
 https://cz.mouser.com/ProductDetail/78-TSDP34138
@@
 Text Notes 14800 4000 0    50   ~ 0
 Akcelerometr\n
-Text Notes 4900 14450 0    50   ~ 0
-Bylo by vhodné připad proudovou ochranu\nsloženou z PTC pojistky a transilu
 Text Label 4300 5400 2    50   ~ 0
 USB_CON+
@@
 Wire Notes Line
 	2200 1450 3850 1450
-Text Notes 2450 15100 0    50   ~ 0
-Je vážný důvod mít jeden senzor na SPI a druhý na I2C?\nPřípadně bych asi očekával, že data z akcelerometru budou\npotřeba s vyšší frekvencí a přesto je na pomalejší sběrnici
 Text Notes 7450 4100 0    50   ~ 0
 Gyroskop\n\n
@@
 BLE MODUL  https://cz.mouser.com/ProductDetail/Microchip-Technology/RN4871-V-RM140?qs=BJlw7L4Cy79E5xvNxQ64Jg%3D%3D
 Wire Notes Line
-	2300 14000 2300 15850
-Wire Notes Line
-	2300 15850 9150 15850
-Wire Notes Line
-	9150 15850 9150 14050
-Wire Notes Line
-	9150 14050 2300 14000
-Text Notes 5250 15550 0    50   ~ 0
-Obecné:\n- Pokud má zapojení jen jednu zem, pak se běžně nepoužívá u značky label GND\n- Schéma by možná bylo lepší pojmout hierarchicky (oddělených částí má docela dost)\n- V případě flat schématu by bylo lepší boxy rozmítit, nějak hezčeji a ne je jen rozházet po prostoru\n- Neexistuje zde jednost v zápisu hodnot: 2k5 vs 2.7k, objevuje se jich zde několik
-Wire Notes Line
-	2300 14300 4300 14300
-Wire Notes Line
-	4300 14300 4300 14000
-Text Notes 2800 14200 0    50   ~ 0
-Užitečné připomínky
-Wire Notes Line
 	7400 7800 21850 7800
 Text Notes 14800 7750 0    50   ~ 0
@@
 	1    11300 9500
 	0    -1   -1   0
-$EndComp
-$Comp
-L SamacSys_Parts:FDD86113LZ Q1
-U 1 1 622E5FCD
-P 4300 12100
-F 0 "Q1" H 4730 12246 50  0000 L CNN
-F 1 "FDD86113LZ" H 4730 12155 50  0000 L CNN
-F 2 "DPAK3-CASE-369AS" H 4750 12050 50  0001 L CNN
-F 3 "https://www.onsemi.com/pub/Collateral/FDD86113LZ-D.pdf" H 4750 11950 50  0001 L CNN
-F 4 "FDD86113LZ N-Channel MOSFET, 5.5 A, 100 V PowerTrench, 3-Pin DPAK ON Semiconductor" H 4750 11850 50  0001 L CNN "Description"
-F 5 "" H 4750 11750 50  0001 L CNN "Height"
-F 6 "512-FDD86113LZ" H 4750 11650 50  0001 L CNN "Mouser Part Number"
-F 7 "https://www.mouser.co.uk/ProductDetail/ON-Semiconductor-Fairchild/FDD86113LZ?qs=Aj0GNA1YSDQLi07jrZVfPw%3D%3D" H 4750 11550 50  0001 L CNN "Mouser Price/Stock"
-F 8 "ON Semiconductor" H 4750 11450 50  0001 L CNN "Manufacturer_Name"
-F 9 "FDD86113LZ" H 4750 11350 50  0001 L CNN "Manufacturer_Part_Number"
-	1    4300 12100
-	1    0    0    -1
 $EndComp
 $Comp
@@
 	1    0    0    -1
 $EndComp
-Text Label 9150 9550 2    50   ~ 0
+Text Label 9100 9700 2    50   ~ 0
 BTN
-$Comp
-L Device:C C23
-U 1 1 6285D17C
-P 8600 9700
-F 0 "C23" H 8715 9746 50  0000 L CNN
-F 1 "100n" H 8715 9655 50  0000 L CNN
-F 2 "Capacitor_SMD:C_0805_2012Metric_Pad1.18x1.45mm_HandSolder" H 8638 9550 50  0001 C CNN
-F 3 "~" H 8600 9700 50  0001 C CNN
-	1    8600 9700
-	1    0    0    -1
-$EndComp
 $Comp
 L Switch:SW_Push_Open SW3
 U 1 1 6285D182
-P 8250 9750
-F 0 "SW3" V 8300 10000 50  0000 R CNN
-F 1 "SW_Push_Open" V 8200 10350 50  0000 R CNN
-F 2 "SamacSys_Parts:PTS815SJM250SMTRLFS" H 8250 9950 50  0001 C CNN
-F 3 "~" H 8250 9950 50  0001 C CNN
-	1    8250 9750
+P 8200 9900
+F 0 "SW3" V 8250 10150 50  0000 R CNN
+F 1 "SW_Push_Open" V 8150 10500 50  0000 R CNN
+F 2 "SamacSys_Parts:PTS815SJM250SMTRLFS" H 8200 10100 50  0001 C CNN
+F 3 "~" H 8200 10100 50  0001 C CNN
+	1    8200 9900
 	0    -1   -1   0
-$EndComp
-$Comp
-L power:GND #PWR0103
-U 1 1 6285D188
-P 8600 10050
-F 0 "#PWR0103" H 8600 9800 50  0001 C CNN
-F 1 "GND" H 8605 9877 50  0001 C CNN
-F 2 "" H 8600 10050 50  0001 C CNN
-F 3 "" H 8600 10050 50  0001 C CNN
-	1    8600 10050
-	1    0    0    -1
 $EndComp
 $Comp
 L power:GND #PWR0104
 U 1 1 6285D18E
-P 8250 10050
-F 0 "#PWR0104" H 8250 9800 50  0001 C CNN
-F 1 "GND" H 8255 9877 50  0001 C CNN
-F 2 "" H 8250 10050 50  0001 C CNN
-F 3 "" H 8250 10050 50  0001 C CNN
-	1    8250 10050
-	1    0    0    -1
-$EndComp
-Wire Wire Line
-	8600 9850 8600 10050
-Wire Wire Line
-	8600 9550 9150 9550
-Wire Wire Line
-	8250 9950 8250 10050
-Wire Wire Line
-	8250 9550 8600 9550
-Connection ~ 8600 9550
+P 8200 10200
+F 0 "#PWR0104" H 8200 9950 50  0001 C CNN
+F 1 "GND" H 8205 10027 50  0001 C CNN
+F 2 "" H 8200 10200 50  0001 C CNN
+F 3 "" H 8200 10200 50  0001 C CNN
+	1    8200 10200
+	1    0    0    -1
+$EndComp
+Wire Wire Line
+	8200 10100 8200 10200
 Text Label 13500 11200 2    50   ~ 0
 BTN
@@
 Text Notes 5600 1500 0    50   ~ 0
 SWD konektor\n\n
+$Comp
+L Device:R R17
+U 1 1 627CCB79
+P 8550 9450
+F 0 "R17" V 8343 9450 50  0000 C CNN
+F 1 "10k" V 8434 9450 50  0000 C CNN
+F 2 "Resistor_SMD:R_0805_2012Metric_Pad1.20x1.40mm_HandSolder" V 8480 9450 50  0001 C CNN
+F 3 "~" H 8550 9450 50  0001 C CNN
+	1    8550 9450
+	1    0    0    1
+$EndComp
+$Comp
+L power:+3.3V #PWR0103
+U 1 1 627CDE79
+P 8550 9200
+F 0 "#PWR0103" H 8550 9050 50  0001 C CNN
+F 1 "+3.3V" H 8565 9373 50  0000 C CNN
+F 2 "" H 8550 9200 50  0001 C CNN
+F 3 "" H 8550 9200 50  0001 C CNN
+	1    8550 9200
+	1    0    0    -1
+$EndComp
+Wire Wire Line
+	8200 9700 8550 9700
+Wire Wire Line
+	8550 9600 8550 9700
+Connection ~ 8550 9700
+Wire Wire Line
+	8550 9700 9100 9700
+Wire Wire Line
+	8550 9300 8550 9200
+$Comp
+L SamacSys_Parts:FDD86113LZ Q1
+U 1 1 622E5FCD
+P 4300 12100
+F 0 "Q1" H 4730 12246 50  0000 L CNN
+F 1 "FDD86113LZ" H 4730 12155 50  0000 L CNN
+F 2 "SamacSys_Parts:DPAK3-CASE-369AS" H 4750 12050 50  0001 L CNN
+F 3 "https://www.onsemi.com/pub/Collateral/FDD86113LZ-D.pdf" H 4750 11950 50  0001 L CNN
+F 4 "FDD86113LZ N-Channel MOSFET, 5.5 A, 100 V PowerTrench, 3-Pin DPAK ON Semiconductor" H 4750 11850 50  0001 L CNN "Description"
+F 5 "" H 4750 11750 50  0001 L CNN "Height"
+F 6 "512-FDD86113LZ" H 4750 11650 50  0001 L CNN "Mouser Part Number"
+F 7 "https://www.mouser.co.uk/ProductDetail/ON-Semiconductor-Fairchild/FDD86113LZ?qs=Aj0GNA1YSDQLi07jrZVfPw%3D%3D" H 4750 11550 50  0001 L CNN "Mouser Price/Stock"
+F 8 "ON Semiconductor" H 4750 11450 50  0001 L CNN "Manufacturer_Name"
+F 9 "FDD86113LZ" H 4750 11350 50  0001 L CNN "Manufacturer_Part_Number"
+	1    4300 12100
+	1    0    0    -1
+$EndComp
 $EndSCHEMATC

Commit message: final_version2_snad
Parts:
- removed FB1: Ferrite_Bead, Resistor_SMD:R_0805_2012Metric_Pad1.20x1.40mm_HandSolder, symbol Device:Ferrite_Bead
- removed J2: Conn_01x02, KICAD_bak:MyConnector2, symbol Connector_Generic:Conn_01x02
- added J2: Conn_01x02_MountingPin, KICAD_bak:Conn01x02_my, symbol Connector_Generic_MountingPin:Conn_01x02_MountingPin
- added R18, R19: 22, Resistor_SMD:R_0603_1608Metric_Pad0.98x0.95mm_HandSolder, symbol Device:R
Connections:
- net GND: now also J1.6 (Shield), J2.MP (MountPin)
- net USB+: now also R19.2; no longer U1.4 (I/O2)
- net USB-: now also R18.1; no longer U1.6 (I/O1)
- net at D2.2 (~~): now also J2.1 (Pin_1)
- net at D2.4 (~~): now also J2.2 (Pin_2)
- new net: R19.1, U1.4 (I/O2)
- new net: R18.2, U1.6 (I/O1)
Other:
- moved on the sheet: U1
Changed lines of the file:
@@
-$EndComp
-$Comp
-L Device:Ferrite_Bead FB1
-U 1 1 62247DD5
-P 3500 6050
-F 0 "FB1" H 3300 6100 50  0000 R CNN
-F 1 "Ferrite_Bead" H 3400 6200 50  0000 R CNN
-F 2 "Resistor_SMD:R_0805_2012Metric_Pad1.20x1.40mm_HandSolder" V 3430 6050 50  0001 C CNN
-F 3 "~" H 3500 6050 50  0001 C CNN
-	1    3500 6050
-	-1   0    0    1
 $EndComp
 $Comp
 L power:GND #PWR04
 U 1 1 622BAF7E
-P 3500 6200
-F 0 "#PWR04" H 3500 5950 50  0001 C CNN
-F 1 "GND" H 3505 6027 50  0001 C CNN
-F 2 "" H 3500 6200 50  0001 C CNN
-F 3 "" H 3500 6200 50  0001 C CNN
-	1    3500 6200
+P 3500 5900
+F 0 "#PWR04" H 3500 5650 50  0001 C CNN
+F 1 "GND" H 3505 5727 50  0001 C CNN
+F 2 "" H 3500 5900 50  0001 C CNN
+F 3 "" H 3500 5900 50  0001 C CNN
+	1    3500 5900
 	1    0    0    -1
 $EndComp
@@
 Wire Notes Line
 	2200 6650 7400 6650
-Text Label 6500 5400 2    50   ~ 0
+Text Label 6900 5250 0    50   ~ 0
 USB+
 $Comp
@@
 Wire Wire Line
 	12250 8600 11700 8600
-$Comp
-L Connector_Generic:Conn_01x02 J2
-U 1 1 61A59630
-P 11500 2700
-F 0 "J2" H 11418 2375 50  0000 C CNN
-F 1 "Conn_01x02" H 11418 2466 50  0000 C CNN
-F 2 "KICAD_bak:MyConnector2" H 11500 2700 50  0001 C CNN
-F 3 "~" H 11500 2700 50  0001 C CNN
-	1    11500 2700
-	-1   0    0    1
-$EndComp
 $Comp
 L power:GND #PWR011
@@
 $EndComp
 Wire Wire Line
-	6050 5400 6500 5400
-Wire Wire Line
-	6050 5600 6500 5600
+	6450 5450 6900 5450
 $Comp
 L Power_Protection:USBLC6-2SC6 U1
 U 1 1 61A7E604
-P 5650 5500
-F 0 "U1" H 5650 4800 50  0000 C CNN
-F 1 "USBLC6-2SC6" H 5650 4900 50  0000 C CNN
-F 2 "Package_TO_SOT_SMD:SOT-23-6" H 5650 5000 50  0001 C CNN
-F 3 "https://www.st.com/resource/en/datasheet/usblc6-2.pdf" H 5850 5850 50  0001 C CNN
-F 4 "https://www.tme.eu/cz/details/usblc6-2sc6/ochranne-diody-site/stmicroelectronics/" H 5650 5500 50  0001 C CNN "Odkaz"
-	1    5650 5500
+P 6050 5350
+F 0 "U1" H 6050 4650 50  0000 C CNN
+F 1 "USBLC6-2SC6" H 6050 4750 50  0000 C CNN
+F 2 "Package_TO_SOT_SMD:SOT-23-6" H 6050 4850 50  0001 C CNN
+F 3 "https://www.st.com/resource/en/datasheet/usblc6-2.pdf" H 6250 5700 50  0001 C CNN
+F 4 "https://www.tme.eu/cz/details/usblc6-2sc6/ochranne-diody-site/stmicroelectronics/" H 6050 5350 50  0001 C CNN "Odkaz"
+	1    6050 5350
 	1    0    0    -1
 $EndComp
@@
 L power:GND #PWR017
 U 1 1 61AE2ED5
-P 5650 5900
-F 0 "#PWR017" H 5650 5650 50  0001 C CNN
-F 1 "GND" H 5655 5727 50  0001 C CNN
-F 2 "" H 5650 5900 50  0001 C CNN
-F 3 "" H 5650 5900 50  0001 C CNN
-	1    5650 5900
+P 6050 5750
+F 0 "#PWR017" H 6050 5500 50  0001 C CNN
+F 1 "GND" H 6055 5577 50  0001 C CNN
+F 2 "" H 6050 5750 50  0001 C CNN
+F 3 "" H 6050 5750 50  0001 C CNN
+	1    6050 5750
 	1    0    0    -1
 $EndComp
@@
 L power:+5V #PWR016
 U 1 1 61AE35A3
-P 5650 5100
-F 0 "#PWR016" H 5650 4950 50  0001 C CNN
-F 1 "+5V" V 5665 5228 50  0000 L CNN
-F 2 "" H 5650 5100 50  0001 C CNN
-F 3 "" H 5650 5100 50  0001 C CNN
-	1    5650 5100
-	1    0    0    -1
-$EndComp
-Text Label 6500 5600 2    50   ~ 0
+P 6050 4950
+F 0 "#PWR016" H 6050 4800 50  0001 C CNN
+F 1 "+5V" V 6065 5078 50  0000 L CNN
+F 2 "" H 6050 4950 50  0001 C CNN
+F 3 "" H 6050 4950 50  0001 C CNN
+	1    6050 4950
+	1    0    0    -1
+$EndComp
+Text Label 6900 5450 2    50   ~ 0
 USB_CON+
-Text Label 4750 5600 0    50   ~ 0
+Text Label 5150 5450 0    50   ~ 0
 USB_CON-
-Text Label 4750 5400 0    50   ~ 0
+Text Label 5150 5250 0    50   ~ 0
 USB-
 Wire Wire Line
-	5250 5600 4750 5600
-Wire Wire Line
-	5250 5400 4750 5400
+	5650 5450 5150 5450
 Text Label 9950 10500 0    50   ~ 0
 SWCLK
@@
 	1    0    0    -1
 $EndComp
+Wire Wire Line
+	6750 5250 6900 5250
+Wire Wire Line
+	5350 5250 5150 5250
+$Comp
+L Device:R R18
+U 1 1 628F3ED9
+P 5500 5250
+F 0 "R18" V 5600 5250 50  0000 C CNN
+F 1 "22" V 5700 5250 50  0000 C CNN
+F 2 "Resistor_SMD:R_0603_1608Metric_Pad0.98x0.95mm_HandSolder" V 5430 5250 50  0001 C CNN
+F 3 "~" H 5500 5250 50  0001 C CNN
+	1    5500 5250
+	0    -1   -1   0
+$EndComp
+$Comp
+L Device:R R19
+U 1 1 628FFF5D
+P 6600 5250
+F 0 "R19" V 6700 5250 50  0000 C CNN
+F 1 "22" V 6800 5250 50  0000 C CNN
+F 2 "Resistor_SMD:R_0603_1608Metric_Pad0.98x0.95mm_HandSolder" V 6530 5250 50  0001 C CNN
+F 3 "~" H 6600 5250 50  0001 C CNN
+	1    6600 5250
+	0    -1   -1   0
+$EndComp
+$Comp
+L Connector_Generic_MountingPin:Conn_01x02_MountingPin J2
+U 1 1 62952341
+P 11500 2700
+F 0 "J2" H 11588 2522 50  0000 L CNN
+F 1 "Conn_01x02_MountingPin" H 11588 2613 50  0000 L CNN
+F 2 "KICAD_bak:Conn01x02_my" H 11500 2700 50  0001 C CNN
+F 3 "~" H 11500 2700 50  0001 C CNN
+	1    11500 2700
+	-1   0    0    1
+$EndComp
+Wire Wire Line
+	11500 2400 11000 2400
+Wire Wire Line
+	11000 2400 11000 3000
+$Comp
+L power:GND #PWR0105
+U 1 1 62983CF7
+P 11000 3000
+F 0 "#PWR0105" H 11000 2750 50  0001 C CNN
+F 1 "GND" H 11005 2827 50  0001 C CNN
+F 2 "" H 11000 3000 50  0001 C CNN
+F 3 "" H 11000 3000 50  0001 C CNN
+	1    11000 3000
+	1    0    0    -1
+$EndComp
