File: bak.sch (KiCad schematic (older format))
At the start: 69 parts, among them CON1 IR_RECIEVER, CON2 HALL_SENSOR1, CON3 HALL_SENSOR2, CON4 SWD, IC1 A3G4250DTR, IC2 MCP112T-195I_TT, IC3 RN4871-V_RM140, IC4 Akcelerometr MC3479, J1 USB_B_Micro, J2 Conn_01x02_MountingPin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

Commit message: final
Parts:
- C12: Umístněí (none) -> Decoupling
- C13, C16, C17, C5, C6, C9: Umístění (none) -> Decoupling
- D1: value D -> NRVS1AFL
- D2: value Usměrňovací můstek ABS210-13 -> ABS210-13
- H1: footprint MountingHole:MountingHole_2.2mm_M2_Pad_Via -> MountingHole:MountingHole_2.7mm_M2.5_Pad_Via
- IC4: value Akcelerometr MC3479 -> MC3479
- J2: value Conn_01x02_MountingPin -> Conn_01x02
- R16: value ? -> 50
Connections:
- net +3.3VA: no longer LDO1.2 (OUTPUT_1), LDO1.4 (OUTPUT_2)
- net GND: no longer LDO1.1 (ADJUST/GROUND)
- net at C18.2, D5.1 (K), D6.1 (K): no longer LDO1.3 (INPUT)
- net MOTOR+ renamed MOTOR_U
- net MOTOR-: no longer names the net of D1.2 (A), J3.2 (Pin_2), Q1.3
- no-connect marks 20 -> 19
Other:
- note added: "Akcelerometr a gyroskop"
- note added: "BLE MODUL\n"
- note added: "Filtrační kondenzátory,\n co nejblíže pinům 1 a 16\n"
- note added: "Filtrační kondeznátory, \nco nejblíže pinu 9"
- note added: "Filtrační kondeznátory, co nejblíže\nk pinům 1, 23, 36, 47,\n"
- note added: "NMOSFET pro ovládání motoru\n\n"
- note added: "Pullup rezistory"
- note added: "Pullup rezistory\n"
- note added: "Signalizační diody"
- note added: "Spínače\n"
- note removed: "ACC https://www.mouser.co.uk/ProductDetail/MEMSIC/MC3479?qs=OlC7AqGiEDmYmlaMvA9fTA%3D%3D"
- note removed: "Akcelerometr\n"
- note removed: "BLE MODUL RN4871-V/RM140"
- note removed: "BLE MODUL https://cz.mouser.com/ProductDetail/Microchip-Technology/RN4871-V-RM140?qs=BJlw7L4Cy79E5xvNxQ64Jg%3D%3D"
- note removed: "Bridge https://www.mouser.co.uk/ProductDetail/Diodes-Incorporated/ABS210-13?qs=5aG0NVq1C4xM%2FxRR9dyQBQ%3D%3D"
- note removed: "Diody pro možnou signalizaci\n"
- note removed: "ESD https://www.tme.eu/cz/details/usblc6-2sc6/ochranne-diody-site/stmicroelectronics/\n"
- note removed: "GYRO https://cz.mouser.com/ProductDetail/511-A3G4250DTR\n"
- note removed: "Gyroskop\n\n"
- note removed: "KRYSTAL https://cz.mouser.com/ProductDetail/ECS/ECS-160-8-36B2-CKM-TR?qs=QNEnbhJQKvaIQPndV3OLHg%3D%3D\n"
- note removed: "LDO https://www.mouser.co.uk/ProductDetail/onsemi/NCP1117ST33T3G?qs=Gev%252BmEvV0iZb%2FE8ahUDx3w%3D%3D"
- note removed: "NMOSFET pro ovládání motoru pomocí PWM\n"
- note removed: "Protection: https://www.mouser.co.uk/ProductDetail/Microchip-Technology/MCP112T-195I-TT?qs=zTHaqZazPEcYKTLEfmIDwg%3D%3D"
- note removed: "Schotky https://cz.mouser.com/ProductDetail/Micro-Commercial-Components-MCC/B5819WS-TP?qs=sGAEpiMZZMuln9v2%2F1E3MaFsjnDe%2F1WFMQWY26r0csM%3D"
- note removed: "USB https://www.mouser.co.uk/ProductDetail/GCT/USB3065-30-00-A?qs=iLbezkQI%252Bshlw4HeJLlWGw%3D%3D"
- note removed: "https://cz.mouser.com/ProductDetail/621-AH49EZ3-G1"
- note removed: "https://cz.mouser.com/ProductDetail/78-TSDP34138"
- note removed: "https://cz.mouser.com/ProductDetail/Wurth-Elektronik/693072010801?qs=7gQLVZk5cPmw4uU1mAcUFg%3D%3D\n"
- moved on the sheet: C1, C10, C11, C12, C13, C14, C15, C16, C17, C18, C19, C2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
